Commit message: urdf: add sonar sensor
Signed-off-by: Thomas Chou <thomas@wytron.com.tw>

File: linorobot2_description/urdf/2wd_properties.urdf.xacro (robot description, xacro)
@@ -20,3 +20,6 @@
     <origin xyz="0.14 0.0 0.045" rpy="0 0 0"/>
   </xacro:property>
+  <xacro:property name="sonar_pose">
+    <origin xyz="0.15 0 0" rpy="0 0 0"/>
+  </xacro:property>
 </robot>

File: linorobot2_description/urdf/4wd_properties.urdf.xacro (robot description, xacro)
@@ -18,3 +18,6 @@
     <origin xyz="-0.065 0 0.255" rpy="0 0 0"/>
   </xacro:property>
+  <xacro:property name="sonar_pose">
+    <origin xyz="0.22 0 0" rpy="0 0 0"/>
+  </xacro:property>
 </robot>

File: linorobot2_description/urdf/mecanum_properties.urdf.xacro (robot description, xacro)
@@ -18,3 +18,6 @@
     <origin xyz="0.2375 0 0.06" rpy="0 0 0"/>
   </xacro:property>
+  <xacro:property name="sonar_pose">
+    <origin xyz="0.22 0 0" rpy="0 0 0"/>
+  </xacro:property>
 </robot>

File: linorobot2_description/urdf/robots/2wd.urdf.xacro (robot description, xacro)
@@ -8,4 +8,5 @@
   <xacro:include filename="$(find linorobot2_description)/urdf/sensors/generic_laser.urdf.xacro" />
   <xacro:include filename="$(find linorobot2_description)/urdf/sensors/depth_sensor.urdf.xacro" />
+  <xacro:include filename="$(find linorobot2_description)/urdf/sensors/sonar.urdf.xacro" />
   <xacro:include filename="$(find linorobot2_description)/urdf/controllers/diff_drive.urdf.xacro" />
   <xacro:base
@@ -60,4 +61,7 @@
     <xacro:insert_block name="depth_sensor_pose" />
   </xacro:depth_sensor>
+  <xacro:sonar>
+    <xacro:insert_block name="sonar_pose" />
+  </xacro:sonar>
   <xacro:diff_drive_controller
     wheel_separation="${wheel_pos_y * 2}"

File: linorobot2_description/urdf/robots/4wd.urdf.xacro (robot description, xacro)
@@ -7,4 +7,5 @@
   <xacro:include filename="$(find linorobot2_description)/urdf/sensors/generic_laser.urdf.xacro" />
   <xacro:include filename="$(find linorobot2_description)/urdf/sensors/depth_sensor.urdf.xacro" />
+  <xacro:include filename="$(find linorobot2_description)/urdf/sensors/sonar.urdf.xacro" />
   <xacro:include filename="$(find linorobot2_description)/urdf/controllers/skid_steer.urdf.xacro" />
   <xacro:base
@@ -59,4 +60,7 @@
     <xacro:insert_block name="depth_sensor_pose" />
   </xacro:depth_sensor>
+  <xacro:sonar>
+    <xacro:insert_block name="sonar_pose" />
+  </xacro:sonar>
   <xacro:diff_drive_controller
     wheel_separation="${wheel_pos_y * 2}"

File: linorobot2_description/urdf/robots/mecanum.urdf.xacro (robot description, xacro)
@@ -7,4 +7,5 @@
   <xacro:include filename="$(find linorobot2_description)/urdf/sensors/generic_laser.urdf.xacro" />
   <xacro:include filename="$(find linorobot2_description)/urdf/sensors/depth_sensor.urdf.xacro" />
+  <xacro:include filename="$(find linorobot2_description)/urdf/sensors/sonar.urdf.xacro" />
   <xacro:include filename="$(find linorobot2_description)/urdf/controllers/omni_drive.urdf.xacro" />
   <xacro:base
@@ -59,4 +60,7 @@
     <xacro:insert_block name="depth_sensor_pose" />
   </xacro:depth_sensor>
+  <xacro:sonar>
+    <xacro:insert_block name="sonar_pose" />
+  </xacro:sonar>
   <xacro:omni_drive_controller/>
 </robot>
